Commit message: Initial commit

File: dist/assets/drone_gripper_1/urdf/drone_gripper_1.urdf (robot description, URDF)
Before this commit: robot drone_gripper_1, 16 links, 15 joints
Links:
- link arm_1: geometry collision mesh filename=package://dist/assets/drone_gripper_1/meshes/arm_1.STL; visual mesh filename=package://dist/assets/drone_gripper_1/meshes/arm_1.STL
- link arm_2: geometry collision mesh filename=package://dist/assets/drone_gripper_1/meshes/arm_2.STL; visual mesh filename=package://dist/assets/drone_gripper_1/meshes/arm_2.STL
- link arm_base: geometry collision mesh filename=package://dist/assets/drone_gripper_1/meshes/arm_base.STL; visual mesh filename=package://dist/assets/drone_gripper_1/meshes/arm_base.STL
- link base: geometry collision mesh filename=package://dist/assets/drone_gripper_1/meshes/base.STL; visual mesh filename=package://dist/assets/drone_gripper_1/meshes/base.STL
- link grip_1: geometry collision mesh filename=package://dist/assets/drone_gripper_1/meshes/grip_1.STL; visual mesh filename=package://dist/assets/drone_gripper_1/meshes/grip_1.STL
- link grip_2: geometry collision mesh filename=package://dist/assets/drone_gripper_1/meshes/grip_2.STL; visual mesh filename=package://dist/assets/drone_gripper_1/meshes/grip_2.STL
- link grip_3: geometry collision mesh filename=package://dist/assets/drone_gripper_1/meshes/grip_3.STL; visual mesh filename=package://dist/assets/drone_gripper_1/meshes/grip_3.STL
- link grip_base: geometry collision mesh filename=package://dist/assets/drone_gripper_1/meshes/grip_base.STL; visual mesh filename=package://dist/assets/drone_gripper_1/meshes/grip_base.STL
- link motor_1: geometry collision mesh filename=package://dist/assets/drone_gripper_1/meshes/motor_1.STL; visual mesh filename=package://dist/assets/drone_gripper_1/meshes/motor_1.STL
- link motor_2: geometry collision mesh filename=package://dist/assets/drone_gripper_1/meshes/motor_2.STL; visual mesh filename=package://dist/assets/drone_gripper_1/meshes/motor_2.STL
- link motor_3: geometry collision mesh filename=package://dist/assets/drone_gripper_1/meshes/motor_3.STL; visual mesh filename=package://dist/assets/drone_gripper_1/meshes/motor_3.STL
- link motor_4: geometry collision mesh filename=package://dist/assets/drone_gripper_1/meshes/motor_4.STL; visual mesh filename=package://dist/assets/drone_gripper_1/meshes/motor_4.STL
- link prop_1: geometry collision mesh filename=package://dist/assets/drone_gripper_1/meshes/prop_1.STL; visual mesh filename=package://dist/assets/drone_gripper_1/meshes/prop_1.STL
- link prop_2: geometry collision mesh filename=package://dist/assets/drone_gripper_1/meshes/prop_2.STL; visual mesh filename=package://dist/assets/drone_gripper_1/meshes/prop_2.STL
- link prop_3: geometry collision mesh filename=package://dist/assets/drone_gripper_1/meshes/prop_3.STL; visual mesh filename=package://dist/assets/drone_gripper_1/meshes/prop_3.STL
- link prop_4: geometry collision mesh filename=package://dist/assets/drone_gripper_1/meshes/prop_4.STL; visual mesh filename=package://dist/assets/drone_gripper_1/meshes/prop_4.STL
